Commit message: spawned robot model in empty sdf

File: src/robot_description/models/robot_fourW/robot_fourW.urdf (robot description, URDF)
Before this commit: robot robot_fourW, 7 links, 6 joints
Links:
- link base_link: mass 0.02494941699556569 -> 5
- link blw: mass 0.0007891680745817908 -> 1
- link brw: mass 0.0007891680745817905 -> 1
- link camera: mass 4.5012174053959215e-06 -> 0.2
- link flw: mass 0.0007891680745817905 -> 1
- link frw: mass 0.0007891680745817905 -> 1
- link lidar: mass 0.0012330751165340462 -> 0.5
Joints:
- joint base_link_joint_blw: axis 0.0 0.0 1.0 -> 4.791376291715144e-32 0.0 1.0; origin xyz=-0.0005000000000000004 0.006012609325439767 0.004039688604814584 rpy=-0.0 -1.5707963267948966 0 -> xyz=-2.2583960717933986 0.9777149358562927 0.4653274178108635 rpy=-1.5707963267948963 1.8735013540549048e-16 4.912736883966281e-15
- joint base_link_joint_brw: axis 0.0 0.0 1.0 -> -4.791376291715144e-32 -0.0 1.0; origin xyz=0.020499999999999997 0.006012609325439767 0.004039688604814584 rpy=-3.141592653589793 -1.5707963267948966 0 -> xyz=-2.2583960717933897 -1.1222850641437068 0.4653274178108629 rpy=1.570796326794897 1.8735013540549048e-16 4.912736883966281e-15
- joint base_link_joint_cam: origin xyz=0.010131079999999999 0.030530519325439764 0.005272178604814584 rpy=-1.5707963267948966 -0.0 0.0 -> xyz=0.19339463820662559 -0.08539349414369497 0.5885762978108627 rpy=-3.1415926535897882 -1.5707963267948957 0
- joint base_link_joint_flw: axis 0.0 0.0 1.0 -> 4.791376291715144e-32 0.0 1.0; origin xyz=-0.0005000000000000004 0.024512609325439767 0.004039688604814584 rpy=-0.0 -1.5707963267948966 0 -> xyz=-0.4083960717933846 0.9777149358563016 0.4653274178108632 rpy=-1.5707963267948963 1.8735013540549048e-16 4.912736883966281e-15
- joint base_link_joint_frw: axis 0.0 0.0 1.0 -> -4.791376291715144e-32 -0.0 1.0; origin xyz=0.020499999999999997 0.024512609325439767 0.004039688604814584 rpy=-3.141592653589793 -1.5707963267948966 0 -> xyz=-0.4083960717933755 -1.1222850641436977 0.4653274178108625 rpy=1.570796326794897 1.8735013540549048e-16 4.912736883966281e-15
- joint base_link_joint_lidar: axis 0.0 0.0 1.0 -> 0.0 4.930380657631324e-32 1.0; origin xyz=0.01 0.014999999325439765 0.008542238604814584 rpy=0.0 -0.0 0.0 -> xyz=-1.359657071793387 -0.07228508414370254 0.9155824778108627 rpy=2.9837243786801003e-16 1.8735013540549048e-16 4.912736883966281e-15
