Commit message: Resolved:added Plugin

File: src/robots_description/models/robot_fourW/robot_fourW.urdf (robot description, URDF)
Before this commit: robot robot_fourW, 7 links, 6 joints
Joints:
- joint base_link_joint_blw: axis 4.791376291715144e-32 0.0 1.0 -> 0 0 1
- joint base_link_joint_brw: axis -4.791376291715144e-32 -0.0 1.0 -> 0 0 -1
- joint base_link_joint_flw: axis 4.791376291715144e-32 0.0 1.0 -> 0 0 1
- joint base_link_joint_frw: axis -4.791376291715144e-32 -0.0 1.0 -> 0 0 -1
